Commit message: organized oh_my_hans robot

File: src/robots/oh_my_hans_description/description/components/elfin10.urdf.xacro (robot description, xacro)
@@ -1,7 +1,7 @@
 <robot
   name="elfin10" xmlns:xacro="http://www.ros.org/wiki/xacro">
-  <xacro:include filename="$(find oh_my_hans_description)/urdf/materials.xacro" />
-  <xacro:include filename="$(find oh_my_hans_description)/urdf/elfin_robot.gazebo" />
-  <xacro:include filename="$(find oh_my_hans_description)/urdf/elfin_transmission.xacro" />
+  <xacro:include filename="$(find oh_my_hans_description)/description/components/materials.xacro" />
+  <xacro:include filename="$(find oh_my_hans_description)/description/components/elfin.gazebo.xacro" />
+  <xacro:include filename="$(find oh_my_hans_description)/description/components/elfin_transmission.xacro" />
   <xacro:property name="PI" value="3.1415926535897931" />
   <xacro:property name="density" value="3.09" />
@@ -38,5 +38,5 @@
       <geometry>
         <mesh
-          filename="$(find oh_my_hans_description)/meshes/elfin_base_link.STL" />
+          filename="$(find oh_my_hans_description)/meshes/elfin/elfin_base_link.stl" />
       </geometry>
       <material
@@ -52,5 +52,5 @@
       <geometry>
         <mesh
-          filename="$(find oh_my_hans_description)/meshes/elfin_base_link.STL" />
+          filename="$(find oh_my_hans_description)/meshes/elfin/elfin_base_link.stl" />
       </geometry>
     </collision>
@@ -78,5 +78,5 @@
       <geometry>
         <mesh
-          filename="$(find oh_my_hans_description)/meshes/elfin_link1.STL" />
+          filename="$(find oh_my_hans_description)/meshes/elfin/elfin_link1.stl" />
       </geometry>
       <material
@@ -92,5 +92,5 @@
       <geometry>
         <mesh
-          filename="$(find oh_my_hans_description)/meshes/elfin_link1.STL" />
+          filename="$(find oh_my_hans_description)/meshes/elfin/elfin_link1.stl" />
       </geometry>
     </collision>
@@ -136,5 +136,5 @@
       <geometry>
         <mesh
-          filename="$(find oh_my_hans_description)/meshes/elfin_link2.STL" />
+          filename="$(find oh_my_hans_description)/meshes/elfin/elfin_link2.stl" />
       </geometry>
       <material
@@ -150,5 +150,5 @@
       <geometry>
         <mesh
-          filename="$(find oh_my_hans_description)/meshes/elfin_link2.STL" />
+          filename="$(find oh_my_hans_description)/meshes/elfin/elfin_link2.stl" />
       </geometry>
     </collision>
@@ -194,5 +194,5 @@
       <geometry>
         <mesh
-          filename="$(find oh_my_hans_description)/meshes/elfin_link3.STL" />
+          filename="$(find oh_my_hans_description)/meshes/elfin/elfin_link3.stl" />
       </geometry>
       <material
@@ -208,5 +208,5 @@
       <geometry>
         <mesh
-          filename="$(find oh_my_hans_description)/meshes/elfin_link3.STL" />
+          filename="$(find oh_my_hans_description)/meshes/elfin/elfin_link3.stl" />
       </geometry>
     </collision>
@@ -252,5 +252,5 @@
       <geometry>
         <mesh
-          filename="$(find oh_my_hans_description)/meshes/elfin_link4.STL" />
+          filename="$(find oh_my_hans_description)/meshes/elfin/elfin_link4.stl" />
       </geometry>
       <material
@@ -266,5 +266,5 @@
       <geometry>
         <mesh
-          filename="$(find oh_my_hans_description)/meshes/elfin_link4.STL" />
+          filename="$(find oh_my_hans_description)/meshes/elfin/elfin_link4.stl" />
       </geometry>
     </collision>
@@ -310,5 +310,5 @@
       <geometry>
         <mesh
-          filename="$(find oh_my_hans_description)/meshes/elfin_link5.STL" />
+          filename="$(find oh_my_hans_description)/meshes/elfin/elfin_link5.stl" />
       </geometry>
       <material
@@ -324,5 +324,5 @@
       <geometry>
         <mesh
-          filename="$(find oh_my_hans_description)/meshes/elfin_link5.STL" />
+          filename="$(find oh_my_hans_description)/meshes/elfin/elfin_link5.stl" />
       </geometry>
     </collision>
@@ -368,5 +368,5 @@
       <geometry>
         <mesh
-          filename="$(find oh_my_hans_description)/meshes/elfin_link6.STL" />
+          filename="$(find oh_my_hans_description)/meshes/elfin/elfin_link6.stl" />
       </geometry>
       <material
@@ -382,5 +382,5 @@
       <geometry>
         <mesh
-          filename="$(find oh_my_hans_description)/meshes/elfin_link6.STL" />
+          filename="$(find oh_my_hans_description)/meshes/elfin/elfin_link6.stl" />
       </geometry>
     </collision>

File: src/robots/oh_my_hans_description/description/components/gripper.urdf.xacro (robot description, xacro)
@@ -18,5 +18,5 @@
       <visual>
         <geometry>
-          <mesh filename="$(find oh_my_hans_description)/meshes/orbbec_camera_mount.stl"
+          <mesh filename="$(find oh_my_hans_description)/meshes/gripper/orbbec_camera_mount.stl"
             scale="1 1 1" />
         </geometry>
@@ -27,5 +27,5 @@
       <collision>
         <geometry>
-          <mesh filename="$(find oh_my_hans_description)/meshes/orbbec_camera_mount.stl"
+          <mesh filename="$(find oh_my_hans_description)/meshes/gripper/orbbec_camera_mount.stl"
             scale="1 1 1" />
         </geometry>
@@ -40,5 +40,5 @@
       <!-- <visual>
         <geometry>
-          <mesh filename="$(find oh_my_hans_description)/meshes/ndt_probe.stl" scale="1 1 1.3" />
+          <mesh filename="$(find oh_my_hans_description)/meshes/gripper/ndt_probe.stl" scale="1 1 1.3" />
         </geometry>
         <material name="Black">
@@ -48,5 +48,5 @@
       <collision>
         <geometry>
-          <mesh filename="$(find oh_my_hans_description)/meshes/ndt_probe.stl" scale="1 1 1.3 " />
+          <mesh filename="$(find oh_my_hans_description)/meshes/gripper/ndt_probe.stl" scale="1 1 1.3 " />
         </geometry>
       </collision> -->

File: src/robots/oh_my_hans_description/description/components/ndt_gripper.urdf.xacro (robot description, xacro)
@@ -22,5 +22,5 @@
       <visual>
         <geometry>
-          <mesh filename="$(find oh_my_hans_description)/meshes/camera_mount.stl" scale="1 1 1" />
+          <mesh filename="$(find oh_my_hans_description)/meshes/gripper/camera_mount.stl" scale="1 1 1" />
         </geometry>
         <material name="LightGrey">
@@ -30,5 +30,5 @@
       <collision>
         <geometry>
-          <mesh filename="$(find oh_my_hans_description)/meshes/camera_mount.stl" scale="1 1 1" />
+          <mesh filename="$(find oh_my_hans_description)/meshes/gripper/camera_mount.stl" scale="1 1 1" />
         </geometry>
       </collision>
@@ -37,5 +37,5 @@
       <visual>
         <geometry>
-          <mesh filename="$(find oh_my_hans_description)/meshes/gripper_ndt.stl" scale="1 1 1" />
+          <mesh filename="$(find oh_my_hans_description)/meshes/gripper/gripper_ndt.stl" scale="1 1 1" />
         </geometry>
         <material name="LightGrey">
@@ -45,5 +45,5 @@
       <collision>
         <geometry>
-          <mesh filename="$(find oh_my_hans_description)/meshes/gripper_ndt.stl" scale="1 1 1 " />
+          <mesh filename="$(find oh_my_hans_description)/meshes/gripper/gripper_ndt.stl" scale="1 1 1 " />
         </geometry>
       </collision>

File: src/robots/oh_my_hans_description/description/components/racer3-wrist.urdf.xacro (robot description, xacro)
@@ -4,9 +4,9 @@
     Author: LMS
    -->
-  <xacro:include filename="$(find oh_my_hans_description)/urdf/common.model.xacro" />
+  <xacro:include filename="$(find oh_my_hans_description)/description/components/common.model.xacro" />
   <xacro:include
-    filename="$(find oh_my_hans_description)/urdf/racer3-wrist.transmission.xacro" />
+    filename="$(find oh_my_hans_description)/description/components/racer3-wrist.transmission.xacro" />
   <xacro:include
-    filename="$(find oh_my_hans_description)/urdf/racer3-wrist.gazebo.xacro" />
+    filename="$(find oh_my_hans_description)/description/components/racer3-wrist.gazebo.xacro" />
   <xacro:macro name="racer3-wrist_robot"
     params="
@@ -31,5 +31,5 @@
         <origin xyz="0 0 0" rpy="0 0 0" />
         <geometry>
-          <mesh filename="$(find oh_my_hans_description)/meshes/base_link.STL" />
+          <mesh filename="$(find oh_my_hans_description)/meshes/racer3/base_link.stl" />
         </geometry>
         <xacro:c_white />
@@ -38,5 +38,5 @@
         <xacro:col_mask_0 />
         <geometry>
-          <mesh filename="$(find oh_my_hans_description)/meshes/base_link.STL" />
+          <mesh filename="$(find oh_my_hans_description)/meshes/racer3/base_link.stl" />
         </geometry>
       </collision>
@@ -52,5 +52,5 @@
         <origin xyz="0 0 0" rpy="0 0 0" />
         <geometry>
-          <mesh filename="$(find oh_my_hans_description)/meshes/Link5.STL" />
+          <mesh filename="$(find oh_my_hans_description)/meshes/racer3/Link5.stl" />
         </geometry>
         <xacro:c_white />
@@ -59,5 +59,5 @@
         <xacro:col_mask_1 />
         <geometry>
-          <mesh filename="$(find oh_my_hans_description)/meshes/Link5.STL" />
+          <mesh filename="$(find oh_my_hans_description)/meshes/racer3/Link5.stl" />
         </geometry>
       </collision>
@@ -73,5 +73,5 @@
         <xacro:c_d_grey />
         <geometry>
-          <mesh filename="$(find oh_my_hans_description)/meshes/Link6.STL" />
+          <mesh filename="$(find oh_my_hans_description)/meshes/racer3/Link6.stl" />
         </geometry>
         <material name="">
@@ -83,5 +83,5 @@
         <xacro:col_mask_0 />
         <geometry>
-          <mesh filename="$(find oh_my_hans_description)/meshes/Link6.STL" />
+          <mesh filename="$(find oh_my_hans_description)/meshes/racer3/Link6.stl" />
         </geometry>
       </collision>

File: src/robots/oh_my_hans_description/description/oh_my_hans_robot.urdf.xacro (robot description, xacro)
@@ -1,7 +1,7 @@
 <robot name="oh_my_hans_robot" xmlns:xacro="http://www.ros.org/wiki/xacro">
   <xacro:property name="robot_namespace" value="oh_my_hans" />
-  <xacro:include filename="$(find oh_my_hans_description)/urdf/elfin10.urdf.xacro" />
-  <xacro:include filename="$(find oh_my_hans_description)/urdf/racer3-wrist.urdf.xacro" />
-  <xacro:include filename="$(find oh_my_hans_description)/urdf/gripper.urdf.xacro" />
+  <xacro:include filename="$(find oh_my_hans_description)/description/components/elfin10.urdf.xacro" />
+  <xacro:include filename="$(find oh_my_hans_description)/description/components/racer3-wrist.urdf.xacro" />
+  <xacro:include filename="$(find oh_my_hans_description)/description/components/gripper.urdf.xacro" />
   <xacro:include filename="$(find orbbec_description)/urdf/femto_bolt.urdf.xacro" />
   <xacro:arg name="kinematics_params"
@@ -21,5 +21,5 @@
     <visual>
       <geometry>
-        <mesh filename="$(find oh_my_hans_description)/meshes/cart.stl" scale="1 1 1" />
+        <mesh filename="$(find oh_my_hans_description)/meshes/cart/cart.stl" scale="1 1 1" />
       </geometry>
       <origin xyz="0.0 0.0 0.0" rpy="0.0 0.0 0" />
@@ -30,5 +30,5 @@
     <collision>
       <geometry>
-        <mesh filename="$(find oh_my_hans_description)/meshes/cart.stl" scale="1 1 1" />
+        <mesh filename="$(find oh_my_hans_description)/meshes/cart/cart.stl" scale="1 1 1" />
       </geometry>
       <origin xyz="0.0 0.0 0.0" rpy="0.0 0.0 0" />
@@ -50,5 +50,5 @@
       <origin xyz="0 0 0" rpy="0 0 0" />
       <geometry>
-        <mesh filename="$(find oh_my_hans_description)/meshes/LIFTKIT_OS_Link1.stl" />
+        <mesh filename="$(find oh_my_hans_description)/meshes/liftkit/LIFTKIT_OS_Link1.stl" />
       </geometry>
       <material name="white" />
@@ -57,5 +57,5 @@
       <origin xyz="0 0 0" rpy="0 0 0" />
       <geometry>
-        <mesh filename="$(find oh_my_hans_description)/meshes/LIFTKIT_OS_Link1.stl" />
+        <mesh filename="$(find oh_my_hans_description)/meshes/liftkit/LIFTKIT_OS_Link1.stl" />
       </geometry>
       <material name="white" />
@@ -77,5 +77,5 @@
       <origin xyz="0 0 0" rpy="0 0 0" />
       <geometry>
-        <mesh filename="$(find oh_my_hans_description)/meshes/LIFTKIT_OS_Link3.stl" />
+        <mesh filename="$(find oh_my_hans_description)/meshes/liftkit/LIFTKIT_OS_Link3.stl" />
       </geometry>
       <material name="white" />
@@ -84,5 +84,5 @@
       <origin xyz="0 0 0" rpy="0 0 0" />
       <geometry>
-        <mesh filename="$(find oh_my_hans_description)/meshes/LIFTKIT_OS_Link3.stl" />
+        <mesh filename="$(find oh_my_hans_description)/meshes/liftkit/LIFTKIT_OS_Link3.stl" />
       </geometry>
       <material name="white" />
@@ -129,5 +129,5 @@
   </link>
   <!-- 8. ROS2 Control Controllers -->
-  <xacro:include filename="$(find oh_my_hans_description)/urdf/arm_topic.ros2_control.xacro" />
+  <xacro:include filename="$(find oh_my_hans_description)/description/components/arm_topic.ros2_control.xacro" />
   <xacro:arm_topic_ros2_control use_fake_hardware="$(arg use_fake_hardware)" sim_gazebo="false"
     sim_ignition="false" />

File: src/robots/oh_my_hans_description/description/racer3-wrist_robot.urdf.xacro (robot description, xacro)
@@ -19,5 +19,5 @@
   <!--load
   racer3-wrist -->
-  <xacro:include filename="$(find oh_my_hans_description)/urdf/racer3-wrist.urdf.xacro" />
+  <xacro:include filename="$(find oh_my_hans_description)/description/components/racer3-wrist.urdf.xacro" />
   <!-- racer3-wrist robot -->
   <xacro:racer3-wrist_robot prefix="$(arg prefix)"
