Commit message: Enh + Fix: nvblox shared setup

File: src/robots/group_a/group_a_description/urdf/group_a_macro.xacro (robot description, xacro)
@@ -1,5 +1,4 @@
 <?xml version="1.0"?>
 <robot xmlns:xacro="http://ros.org">
-    <!-- Ορισμός του Macro: group_a_robot -->
     <xacro:macro name="group_a_robot"
         params="
@@ -7,7 +6,5 @@
         namespace='group_a'
         lift_type='ur_620'
-        lift_prefix='lift_'
         ur_type='ur10'
-        ur_prefix='ur_'
         sim_gazebo='true'
         use_fake_hardware='false'
@@ -15,9 +12,20 @@
         *origin"
     >
+        <!-- ── Derived prefixes from namespace ──────────────────────────────────
+             All links/joints in the kinematic chain get the namespace prefix.
+             This ensures each robot has a unique TF tree rooted at world.
+             lift_prefix : e.g. "robot_1/lift_"
+             ur_prefix   : e.g. "robot_1/ur_"
+        ──────────────────────────────────────────────────────────────────────── -->
+        <xacro:property name="lift_prefix" value="${namespace}/lift_" />
+        <xacro:property name="ur_prefix" value="${namespace}/ur_" />
         <!-- === Includes === -->
         <xacro:include filename="$(find ewellix_description)/urdf/ewellix_macro.xacro" />
         <xacro:include filename="$(find ur_description)/urdf/ur_macro.xacro" />
         <xacro:include filename="$(find ur_description)/urdf/inc/ur_joint_control.xacro" />
-        <!-- === Ewellix Lift === -->
+        <!-- === Ewellix Lift ────────────────────────────────────────────────────
+             tf_prefix="${lift_prefix}" → all lift links become robot_1/lift_*
+             parent stays "world" (unprefixed global anchor)
+        ──────────────────────────────────────────────────────────────────────── -->
         <xacro:ewellix_lift
             parent="${parent}"
@@ -32,5 +40,8 @@
             <xacro:insert_block name="origin" />
         </xacro:ewellix_lift>
-        <!-- === UR Arm (mounted on ewellix top) === -->
+        <!-- === UR Arm ──────────────────────────────────────────────────────────
+             tf_prefix="${ur_prefix}"       → all UR links become robot_1/ur_*
+             parent="${lift_prefix}mount"   → robot_1/lift_mount
+        ──────────────────────────────────────────────────────────────────────── -->
         <xacro:ur_robot
             name="${namespace}_${ur_type}"
@@ -44,5 +55,5 @@
             <origin xyz="0 0 0" rpy="0 0 0" />
         </xacro:ur_robot>
-        <!-- UR ros2_control block (Διορθωμένο Όνομα Υλικού) -->
+        <!-- === UR ros2_control block ─────────────────────────────────────────── -->
         <ros2_control name="${namespace}_${ur_type}_hardware" type="system">
             <hardware>
@@ -56,6 +67,9 @@
             <xacro:ur_joint_control_description tf_prefix="${ur_prefix}" />
         </ros2_control>
-        <!-- === Orbbec Camera at UR end-effector (Διορθωμένα Ονόματα) === -->
-        <link name="${namespace}_camera_link">
+        <!-- === Camera at UR end-effector ──────────────────────────────────────
+             Link names: ${namespace}/camera_link  →  e.g. robot_1/camera_link
+             Parent:     ${ur_prefix}tool0         →  e.g. robot_1/ur_tool0
+        ──────────────────────────────────────────────────────────────────────── -->
+        <link name="${namespace}/camera_link">
             <visual>
                 <geometry>
@@ -77,17 +91,17 @@
             </inertial>
         </link>
-        <joint name="${namespace}_camera_joint" type="fixed">
-            <parent link="${ur_prefix}tool0" />
-            <child link="${namespace}_camera_link" />
+        <joint name="${namespace}/camera_joint" type="fixed">
+            <parent link="${ur_prefix}tool0" />          <!-- robot_1/ur_tool0 -->
+            <child link="${namespace}/camera_link" />   <!-- robot_1/camera_link -->
             <origin xyz="0 0 0.020" rpy="0 0 0" />
         </joint>
         <!-- Optical frame -->
-        <link name="${namespace}_camera_optical_frame" />
-        <joint name="${namespace}_camera_optical_joint" type="fixed">
-            <parent link="${namespace}_camera_link" />
-            <child link="${namespace}_camera_optical_frame" />
+        <link name="${namespace}/camera_optical_frame" />
+        <joint name="${namespace}/camera_optical_joint" type="fixed">
+            <parent link="${namespace}/camera_link" />
+            <child link="${namespace}/camera_optical_frame" />
             <origin xyz="0 0 0" rpy="${-pi/2} 0 ${-pi/2}" />
         </joint>
-        <!-- === Gazebo-only blocks === -->
+        <!-- === Gazebo-only blocks ──────────────────────────────────────────── -->
         <xacro:if value="${sim_gazebo}">
             <gazebo>
@@ -110,5 +124,5 @@
             </gazebo>
             <!-- Orbbec RGBD sensor -->
-            <gazebo reference="${namespace}_camera_link">
+            <gazebo reference="${namespace}/camera_link">
                 <sensor name="${namespace}_orbbec_camera" type="rgbd_camera">
                     <camera>
@@ -128,5 +142,5 @@
                             <stddev>0.007</stddev>
                         </noise>
-                        <optical_frame_id>${namespace}_camera_optical_frame</optical_frame_id>
+                        <optical_frame_id>${namespace}/camera_optical_frame</optical_frame_id>
                     </camera>
                     <always_on>1</always_on>
