Commit message: Fix: working rviz and moveit planning - Issues with ewellix start state

File: src/robots/group_a/group_a_description/urdf/group_a_macro.xacro (robot description, xacro)
@@ -39,4 +39,5 @@
             use_fake_hardware="${use_fake_hardware}"
             sim_gazebo="${sim_gazebo}"
+            initial_positions="${dict(upper=0.0, lower=0.0)}"
         >
             <xacro:insert_block name="origin" />

File: src/robots/group_a/group_a_moveit_config/config/combined_system.ros2_control.xacro (robot description, xacro)
@@ -2,5 +2,6 @@
 <robot xmlns:xacro="http://www.ros.org/wiki/xacro">
     <xacro:macro name="combined_system_ros2_control" params="name initial_positions_file">
-        <xacro:property name="initial_positions" value="${xacro.load_yaml(initial_positions_file)['initial_positions']}"/>
+        <xacro:property name="initial_positions"
+            value="${xacro.load_yaml(initial_positions_file)['initial_positions']}" />
         <ros2_control name="${name}" type="system">
             <hardware>
@@ -9,51 +10,51 @@
             </hardware>
             <joint name="lift_lower_joint">
-                <command_interface name="position"/>
+                <command_interface name="position" />
                 <state_interface name="position">
-                  <param name="initial_value">${initial_positions['lift_lower_joint']}</param>
+                    <param name="initial_value">${initial_positions['lift_lower_joint']}</param>
                 </state_interface>
-                <state_interface name="velocity"/>
+                <state_interface name="velocity" />
             </joint>
             <joint name="ur_shoulder_pan_joint">
-                <command_interface name="position"/>
+                <command_interface name="position" />
                 <state_interface name="position">
-                  <param name="initial_value">${initial_positions['ur_shoulder_pan_joint']}</param>
+                    <param name="initial_value">${initial_positions['ur_shoulder_pan_joint']}</param>
                 </state_interface>
-                <state_interface name="velocity"/>
+                <state_interface name="velocity" />
             </joint>
             <joint name="ur_shoulder_lift_joint">
-                <command_interface name="position"/>
+                <command_interface name="position" />
                 <state_interface name="position">
-                  <param name="initial_value">${initial_positions['ur_shoulder_lift_joint']}</param>
+                    <param name="initial_value">${initial_positions['ur_shoulder_lift_joint']}</param>
                 </state_interface>
-                <state_interface name="velocity"/>
+                <state_interface name="velocity" />
             </joint>
             <joint name="ur_elbow_joint">
-                <command_interface name="position"/>
+                <command_interface name="position" />
                 <state_interface name="position">
-                  <param name="initial_value">${initial_positions['ur_elbow_joint']}</param>
+                    <param name="initial_value">${initial_positions['ur_elbow_joint']}</param>
                 </state_interface>
-                <state_interface name="velocity"/>
+                <state_interface name="velocity" />
             </joint>
             <joint name="ur_wrist_1_joint">
-                <command_interface name="position"/>
+                <command_interface name="position" />
                 <state_interface name="position">
-                  <param name="initial_value">${initial_positions['ur_wrist_1_joint']}</param>
+                    <param name="initial_value">${initial_positions['ur_wrist_1_joint']}</param>
                 </state_interface>
-                <state_interface name="velocity"/>
+                <state_interface name="velocity" />
             </joint>
             <joint name="ur_wrist_2_joint">
-                <command_interface name="position"/>
+                <command_interface name="position" />
                 <state_interface name="position">
-                  <param name="initial_value">${initial_positions['ur_wrist_2_joint']}</param>
+                    <param name="initial_value">${initial_positions['ur_wrist_2_joint']}</param>
                 </state_interface>
-                <state_interface name="velocity"/>
+                <state_interface name="velocity" />
             </joint>
             <joint name="ur_wrist_3_joint">
-                <command_interface name="position"/>
+                <command_interface name="position" />
                 <state_interface name="position">
-                  <param name="initial_value">${initial_positions['ur_wrist_3_joint']}</param>
+                    <param name="initial_value">${initial_positions['ur_wrist_3_joint']}</param>
                 </state_interface>
-                <state_interface name="velocity"/>
+                <state_interface name="velocity" />
             </joint>
         </ros2_control>

Commit message: FIx: resolved ewelix start state issue
moved the ros2 control block into the main composition xacro instead of reling on auto generated from the package

File: src/robots/group_a/group_a_description/urdf/group_a_macro.xacro (robot description, xacro)
@@ -1,4 +1,4 @@
 <?xml version="1.0"?>
-<robot xmlns:xacro="http://ros.org">
+<robot xmlns:xacro="http://www.ros.org/wiki/xacro">
     <xacro:macro name="group_a_robot"
         params="
@@ -36,11 +36,52 @@
             add_mount="true"
             parameters_file="$(find ewellix_description)/config/${lift_type}.yaml"
-            generate_ros2_control_tag="true"
+            generate_ros2_control_tag="false"
             use_fake_hardware="${use_fake_hardware}"
             sim_gazebo="${sim_gazebo}"
-            initial_positions="${dict(upper=0.0, lower=0.0)}"
         >
             <xacro:insert_block name="origin" />
         </xacro:ewellix_lift>
+        <xacro:property name="parameters_file"
+            value="$(find ewellix_description)/config/${lift_type}.yaml" />
+        <xacro:property name="parameters"
+            value="${xacro.load_yaml(parameters_file)}" />
+        <!-- ROS 2 Controls -->
+        <ros2_control name="${tf_prefix}hardware" type="system">
+            <hardware>
+                <xacro:if value="${sim_gazebo}">
+                    <plugin>gz_ros2_control/GazeboSimSystem</plugin>
+                </xacro:if>
+                <xacro:if value="${use_fake_hardware}">
+                    <plugin>mock_components/GenericSystem</plugin>
+                    <param name="state_following_offset">0.0</param>
+                    <param name="calculate_dynamics">true</param>
+                </xacro:if>
+                <xacro:unless value="${use_fake_hardware or sim_gazebo}">
+                    <plugin>ewellix_driver/EwellixHardwareInterface</plugin>
+                    <param name="port">${port}</param>
+                    <param name="baud">${baud}</param>
+                    <param name="timeout">${timeout}</param>
+                    <param name="conversion">${conversion}</param>
+                    <param name="rated_effort">${rated_effort}</param>
+                    <param name="tolerance">${tolerance}</param>
+                    <param name="encoder_limits_lower">${parameters.encoder_limits.lower}</param>
+                    <param name="encoder_limits_upper">${parameters.encoder_limits.upper}</param>
+                </xacro:unless>
+            </hardware>
+            <joint name="${lift_prefix}lower_joint">
+                <command_interface name="position" />
+                <state_interface name="position">
+                    <param name="initial_value">${parameters.lower.joint.limit.lower + 0.001}</param>
+                </state_interface>
+                <state_interface name="velocity" />
+                <state_interface name="effort" />
+            </joint>
+            <xacro:if value="${sim_gazebo or use_fake_hardware}">
+                <joint name="${lift_prefix}upper_joint">
+                    <param name="mimic">${lift_prefix}lower_joint</param>
+                    <param name="multiplier">1</param>
+                </joint>
+            </xacro:if>
+        </ros2_control>
         <!-- === UR Arm ──────────────────────────────────────────────────────────
              prefix="${ur_prefix}"       → all UR links become robot_1/ur_*
