Commit message: TMP - todo not working sdrf namespaces in moveit movegroup node

File: src/robots/group_a/group_a_description/config/combined_system.srdf.xacro (robot description, xacro)
@@ -5,62 +5,56 @@
     src/robots/group_a/group_a_moveit_config/config/combined_system.srdf
 -->
-<robot xmlns:xacro="http://ros.org" name="combined_system">
+<robot xmlns:xacro="http://ros.org/xacro" name="combined_system">
     <!-- Ορισμός παραμέτρου prefix (κενό ως προεπιλογή) -->
-    <xacro:arg name="prefix" default="" />
-    <xacro:property name="p" value="$(arg prefix)" />
+    <xacro:arg name="tf_prefix" default="" />
+    <group name="all">
+        <chain base_link="$(arg tf_prefix)lift_base_link" tip_link="$(arg tf_prefix)ur_ft_frame"/>
+    </group>
     <group name="lift">
-        <chain base_link="${p}lift_base_link" tip_link="${p}lift_mount_link" />
+        <chain base_link="$(arg tf_prefix)lift_base_link" tip_link="$(arg tf_prefix)lift_mount"/>
     </group>
     <group name="ur">
-        <chain base_link="${p}ur_base_link" tip_link="${p}ur_ft_frame" />
+        <chain base_link="$(arg tf_prefix)ur_base_link" tip_link="$(arg tf_prefix)ur_ft_frame"/>
     </group>
-    <group name="all">
-        <chain base_link="${p}lift_base_link" tip_link="${p}ur_ft_frame" />
-    </group>
-    <virtual_joint name="world_joint" type="fixed" parent_frame="world"
-        child_link="${p}lift_base_link" />
-    <!-- DISABLE COLLISIONS -->
-    <disable_collisions link1="${p}group_a_camera_link" link2="${p}ur_wrist_1_link" reason="Never" />
-    <disable_collisions link1="${p}group_a_camera_link" link2="${p}ur_wrist_2_link" reason="Never" />
-    <disable_collisions link1="${p}group_a_camera_link" link2="${p}ur_wrist_3_link"
-        reason="Adjacent" />
-    <disable_collisions link1="${p}lift_base_link" link2="${p}lift_lower_link" reason="Adjacent" />
-    <disable_collisions link1="${p}lift_base_link" link2="${p}lift_mount_link" reason="Never" />
-    <disable_collisions link1="${p}lift_base_link" link2="${p}lift_plate_link" reason="Adjacent" />
-    <disable_collisions link1="${p}lift_base_link" link2="${p}lift_upper_link" reason="Default" />
-    <disable_collisions link1="${p}lift_base_link" link2="${p}ur_base_link_inertia" reason="Never" />
-    <disable_collisions link1="${p}lift_base_link" link2="${p}ur_shoulder_link" reason="Never" />
-    <disable_collisions link1="${p}lift_lower_link" link2="${p}lift_mount_link" reason="Never" />
-    <disable_collisions link1="${p}lift_lower_link" link2="${p}lift_plate_link" reason="Never" />
-    <disable_collisions link1="${p}lift_lower_link" link2="${p}lift_upper_link" reason="Adjacent" />
-    <disable_collisions link1="${p}lift_lower_link" link2="${p}ur_base_link_inertia" reason="Never" />
-    <disable_collisions link1="${p}lift_lower_link" link2="${p}ur_shoulder_link" reason="Never" />
-    <disable_collisions link1="${p}lift_lower_link" link2="${p}ur_upper_arm_link" reason="Never" />
-    <disable_collisions link1="${p}lift_mount_link" link2="${p}lift_plate_link" reason="Never" />
-    <disable_collisions link1="${p}lift_mount_link" link2="${p}lift_upper_link" reason="Adjacent" />
-    <disable_collisions link1="${p}lift_mount_link" link2="${p}ur_base_link_inertia"
-        reason="Adjacent" />
-    <disable_collisions link1="${p}lift_mount_link" link2="${p}ur_shoulder_link" reason="Never" />
-    <disable_collisions link1="${p}lift_plate_link" link2="${p}lift_upper_link" reason="Never" />
-    <disable_collisions link1="${p}lift_plate_link" link2="${p}ur_base_link_inertia" reason="Never" />
-    <disable_collisions link1="${p}lift_plate_link" link2="${p}ur_shoulder_link" reason="Never" />
-    <disable_collisions link1="${p}lift_plate_link" link2="${p}ur_upper_arm_link" reason="Never" />
-    <disable_collisions link1="${p}lift_upper_link" link2="${p}ur_base_link_inertia" reason="Never" />
-    <disable_collisions link1="${p}lift_upper_link" link2="${p}ur_shoulder_link" reason="Never" />
-    <disable_collisions link1="${p}lift_upper_link" link2="${p}ur_upper_arm_link" reason="Never" />
-    <disable_collisions link1="${p}lift_upper_link" link2="${p}ur_wrist_1_link" reason="Never" />
-    <disable_collisions link1="${p}ur_base_link_inertia" link2="${p}ur_shoulder_link"
-        reason="Adjacent" />
-    <disable_collisions link1="${p}ur_base_link_inertia" link2="${p}ur_upper_arm_link"
-        reason="Never" />
-    <disable_collisions link1="${p}ur_base_link_inertia" link2="${p}ur_wrist_1_link" reason="Never" />
-    <disable_collisions link1="${p}ur_base_link_inertia" link2="${p}ur_wrist_2_link" reason="Never" />
-    <disable_collisions link1="${p}ur_forearm_link" link2="${p}ur_upper_arm_link" reason="Adjacent" />
-    <disable_collisions link1="${p}ur_forearm_link" link2="${p}ur_wrist_1_link" reason="Adjacent" />
-    <disable_collisions link1="${p}ur_shoulder_link" link2="${p}ur_upper_arm_link" reason="Adjacent" />
-    <disable_collisions link1="${p}ur_shoulder_link" link2="${p}ur_wrist_1_link" reason="Never" />
-    <disable_collisions link1="${p}ur_shoulder_link" link2="${p}ur_wrist_2_link" reason="Never" />
-    <disable_collisions link1="${p}ur_wrist_1_link" link2="${p}ur_wrist_2_link" reason="Adjacent" />
-    <disable_collisions link1="${p}ur_wrist_1_link" link2="${p}ur_wrist_3_link" reason="Never" />
-    <disable_collisions link1="${p}ur_wrist_2_link" link2="${p}ur_wrist_3_link" reason="Adjacent" />
+    <!--VIRTUAL JOINT: Purpose: this element defines a virtual joint between a robot link and an external frame of reference (considered fixed with respect to the robot)-->
+    <virtual_joint name="world_joint" type="fixed" parent_frame="world" child_link="$(arg tf_prefix)lift_base_link"/>
+    <!--DISABLE COLLISIONS: By default it is assumed that any link of the robot could potentially come into collision with any other link in the robot. This tag disables collision checking between a specified pair of links. -->
+    <disable_collisions link1="$(arg tf_prefix)camera_link" link2="$(arg tf_prefix)ur_wrist_1_link" reason="Never"/>
+    <disable_collisions link1="$(arg tf_prefix)camera_link" link2="$(arg tf_prefix)ur_wrist_2_link" reason="Never"/>
+    <disable_collisions link1="$(arg tf_prefix)camera_link" link2="$(arg tf_prefix)ur_wrist_3_link" reason="Adjacent"/>
+    <disable_collisions link1="$(arg tf_prefix)lift_base_link" link2="$(arg tf_prefix)lift_lower_link" reason="Adjacent"/>
+    <disable_collisions link1="$(arg tf_prefix)lift_base_link" link2="$(arg tf_prefix)lift_mount_link" reason="Never"/>
+    <disable_collisions link1="$(arg tf_prefix)lift_base_link" link2="$(arg tf_prefix)lift_plate_link" reason="Adjacent"/>
+    <disable_collisions link1="$(arg tf_prefix)lift_base_link" link2="$(arg tf_prefix)lift_upper_link" reason="Default"/>
+    <disable_collisions link1="$(arg tf_prefix)lift_base_link" link2="$(arg tf_prefix)ur_base_link_inertia" reason="Never"/>
+    <disable_collisions link1="$(arg tf_prefix)lift_base_link" link2="$(arg tf_prefix)ur_shoulder_link" reason="Never"/>
+    <disable_collisions link1="$(arg tf_prefix)lift_lower_link" link2="$(arg tf_prefix)lift_mount_link" reason="Never"/>
+    <disable_collisions link1="$(arg tf_prefix)lift_lower_link" link2="$(arg tf_prefix)lift_plate_link" reason="Never"/>
+    <disable_collisions link1="$(arg tf_prefix)lift_lower_link" link2="$(arg tf_prefix)lift_upper_link" reason="Adjacent"/>
+    <disable_collisions link1="$(arg tf_prefix)lift_lower_link" link2="$(arg tf_prefix)ur_base_link_inertia" reason="Never"/>
+    <disable_collisions link1="$(arg tf_prefix)lift_lower_link" link2="$(arg tf_prefix)ur_shoulder_link" reason="Never"/>
+    <disable_collisions link1="$(arg tf_prefix)lift_lower_link" link2="$(arg tf_prefix)ur_upper_arm_link" reason="Never"/>
+    <disable_collisions link1="$(arg tf_prefix)lift_mount_link" link2="$(arg tf_prefix)lift_plate_link" reason="Never"/>
+    <disable_collisions link1="$(arg tf_prefix)lift_mount_link" link2="$(arg tf_prefix)lift_upper_link" reason="Adjacent"/>
+    <disable_collisions link1="$(arg tf_prefix)lift_mount_link" link2="$(arg tf_prefix)ur_base_link_inertia" reason="Adjacent"/>
+    <disable_collisions link1="$(arg tf_prefix)lift_mount_link" link2="$(arg tf_prefix)ur_shoulder_link" reason="Never"/>
+    <disable_collisions link1="$(arg tf_prefix)lift_plate_link" link2="$(arg tf_prefix)lift_upper_link" reason="Never"/>
+    <disable_collisions link1="$(arg tf_prefix)lift_plate_link" link2="$(arg tf_prefix)ur_base_link_inertia" reason="Never"/>
+    <disable_collisions link1="$(arg tf_prefix)lift_plate_link" link2="$(arg tf_prefix)ur_shoulder_link" reason="Never"/>
+    <disable_collisions link1="$(arg tf_prefix)lift_plate_link" link2="$(arg tf_prefix)ur_upper_arm_link" reason="Never"/>
+    <disable_collisions link1="$(arg tf_prefix)lift_upper_link" link2="$(arg tf_prefix)ur_base_link_inertia" reason="Never"/>
+    <disable_collisions link1="$(arg tf_prefix)lift_upper_link" link2="$(arg tf_prefix)ur_shoulder_link" reason="Never"/>
+    <disable_collisions link1="$(arg tf_prefix)lift_upper_link" link2="$(arg tf_prefix)ur_upper_arm_link" reason="Never"/>
+    <disable_collisions link1="$(arg tf_prefix)lift_upper_link" link2="$(arg tf_prefix)ur_wrist_1_link" reason="Never"/>
+    <disable_collisions link1="$(arg tf_prefix)ur_base_link_inertia" link2="$(arg tf_prefix)ur_shoulder_link" reason="Adjacent"/>
+    <disable_collisions link1="$(arg tf_prefix)ur_base_link_inertia" link2="$(arg tf_prefix)ur_upper_arm_link" reason="Never"/>
+    <disable_collisions link1="$(arg tf_prefix)ur_base_link_inertia" link2="$(arg tf_prefix)ur_wrist_1_link" reason="Never"/>
+    <disable_collisions link1="$(arg tf_prefix)ur_forearm_link" link2="$(arg tf_prefix)ur_upper_arm_link" reason="Adjacent"/>
+    <disable_collisions link1="$(arg tf_prefix)ur_forearm_link" link2="$(arg tf_prefix)ur_wrist_1_link" reason="Adjacent"/>
+    <disable_collisions link1="$(arg tf_prefix)ur_shoulder_link" link2="$(arg tf_prefix)ur_upper_arm_link" reason="Adjacent"/>
+    <disable_collisions link1="$(arg tf_prefix)ur_shoulder_link" link2="$(arg tf_prefix)ur_wrist_1_link" reason="Never"/>
+    <disable_collisions link1="$(arg tf_prefix)ur_shoulder_link" link2="$(arg tf_prefix)ur_wrist_2_link" reason="Never"/>
+    <disable_collisions link1="$(arg tf_prefix)ur_wrist_1_link" link2="$(arg tf_prefix)ur_wrist_2_link" reason="Adjacent"/>
+    <disable_collisions link1="$(arg tf_prefix)ur_wrist_1_link" link2="$(arg tf_prefix)ur_wrist_3_link" reason="Never"/>
+    <disable_collisions link1="$(arg tf_prefix)ur_wrist_2_link" link2="$(arg tf_prefix)ur_wrist_3_link" reason="Adjacent"/>
 </robot>

File: src/robots/group_a/group_a_description/urdf/group_a.urdf.xacro (robot description, xacro)
@@ -1,4 +1,4 @@
 <?xml version="1.0"?>
-<robot name="combined_system" xmlns:xacro="http://ros.org">
+<robot name="combined_system" xmlns:xacro="http://ros.org/xacro">
   <!-- 1. Δήλωση των Arguments που γίνονται inject από το Launch Setup -->
   <xacro:arg name="parent" default="world" />
@@ -9,5 +9,6 @@
   <xacro:arg name="sim_gazebo" default="false" />
   <xacro:arg name="use_fake_hardware" default="true" />
-  <xacro:arg name="namespace" default="group_a" />
+  <xacro:arg name="tf_prefix" default="" />
+  <xacro:arg name="namespace" default="" />
   <xacro:arg name="simulation_controllers"
     default='$(find group_a_bringup)/config/controllers.yaml' />
@@ -25,4 +26,5 @@
     sim_gazebo="$(arg sim_gazebo)"
     use_fake_hardware="$(arg use_fake_hardware)"
+    tf_prefix="$(arg tf_prefix)"
     namespace="$(arg namespace)"
     simulation_controllers="$(arg simulation_controllers)"

File: src/robots/group_a/group_a_description/urdf/group_a_macro.xacro (robot description, xacro)
@@ -4,5 +4,6 @@
         params="
         parent
-        namespace='group_a'
+        tf_prefix=''
+        namespace=''
         lift_type='ur_620'
         ur_type='ur10'
@@ -18,6 +19,7 @@
              ur_prefix   : e.g. "robot_1/ur_"
         ──────────────────────────────────────────────────────────────────────── -->
-        <xacro:property name="lift_prefix" value="${namespace}/lift_" />
-        <xacro:property name="ur_prefix" value="${namespace}/ur_" />
+        <xacro:property name="prefix" value="${namespace}/${tf_prefix}" />
+        <xacro:property name="lift_prefix" value="${prefix}lift_" />
+        <xacro:property name="ur_prefix" value="${prefix}ur_" />
         <!-- === Includes === -->
         <xacro:include filename="$(find ewellix_description)/urdf/ewellix_macro.xacro" />
@@ -25,5 +27,5 @@
         <xacro:include filename="$(find ur_description)/urdf/inc/ur_joint_control.xacro" />
         <!-- === Ewellix Lift ────────────────────────────────────────────────────
-             tf_prefix="${lift_prefix}" → all lift links become robot_1/lift_*
+             prefix="${lift_prefix}" → all lift links become robot_1/lift_*
              parent stays "world" (unprefixed global anchor)
         ──────────────────────────────────────────────────────────────────────── -->
@@ -41,9 +43,9 @@
         </xacro:ewellix_lift>
         <!-- === UR Arm ──────────────────────────────────────────────────────────
-             tf_prefix="${ur_prefix}"       → all UR links become robot_1/ur_*
+             prefix="${ur_prefix}"       → all UR links become robot_1/ur_*
              parent="${lift_prefix}mount"   → robot_1/lift_mount
         ──────────────────────────────────────────────────────────────────────── -->
         <xacro:ur_robot
-            name="${namespace}_${ur_type}"
+            name="${ur_type}"
             tf_prefix="${ur_prefix}"
             parent="${lift_prefix}mount"
@@ -56,5 +58,5 @@
         </xacro:ur_robot>
         <!-- === UR ros2_control block ─────────────────────────────────────────── -->
-        <ros2_control name="${namespace}_${ur_type}_hardware" type="system">
+        <ros2_control name="${prefix}${ur_type}_hardware" type="system">
             <hardware>
                 <xacro:if value="${sim_gazebo}">
@@ -68,8 +70,8 @@
         </ros2_control>
         <!-- === Camera at UR end-effector ──────────────────────────────────────
-             Link names: ${namespace}/camera_link  →  e.g. robot_1/camera_link
+             Link names: ${prefix}camera_link  →  e.g. robot_1/camera_link
              Parent:     ${ur_prefix}tool0         →  e.g. robot_1/ur_tool0
         ──────────────────────────────────────────────────────────────────────── -->
-        <link name="${namespace}/camera_link">
+        <link name="${prefix}camera_link">
             <visual>
                 <geometry>
@@ -91,14 +93,14 @@
             </inertial>
         </link>
-        <joint name="${namespace}/camera_joint" type="fixed">
+        <joint name="${prefix}camera_joint" type="fixed">
             <parent link="${ur_prefix}tool0" />          <!-- robot_1/ur_tool0 -->
-            <child link="${namespace}/camera_link" />   <!-- robot_1/camera_link -->
+            <child link="${prefix}camera_link" />   <!-- robot_1/camera_link -->
             <origin xyz="0 0 0.020" rpy="0 0 0" />
         </joint>
         <!-- Optical frame -->
-        <link name="${namespace}/camera_optical_frame" />
-        <joint name="${namespace}/camera_optical_joint" type="fixed">
-            <parent link="${namespace}/camera_link" />
-            <child link="${namespace}/camera_optical_frame" />
+        <link name="${prefix}camera_optical_frame" />
+        <joint name="${prefix}camera_optical_joint" type="fixed">
+            <parent link="${prefix}camera_link" />
+            <child link="${prefix}camera_optical_frame" />
             <origin xyz="0 0 0" rpy="${-pi/2} 0 ${-pi/2}" />
         </joint>
@@ -124,6 +126,6 @@
             </gazebo>
             <!-- Orbbec RGBD sensor -->
-            <gazebo reference="${namespace}/camera_link">
-                <sensor name="${namespace}_orbbec_camera" type="rgbd_camera">
+            <gazebo reference="${prefix}camera_link">
+                <sensor name="${prefix}orbbec_camera" type="rgbd_camera">
                     <camera>
                         <horizontal_fov>1.2120256</horizontal_fov>
@@ -142,10 +144,10 @@
                             <stddev>0.007</stddev>
                         </noise>
-                        <optical_frame_id>${namespace}/camera_optical_frame</optical_frame_id>
+                        <optical_frame_id>${prefix}camera_optical_frame</optical_frame_id>
                     </camera>
                     <always_on>1</always_on>
                     <update_rate>10</update_rate>
                     <visualize>false</visualize>
-                    <topic>/${namespace}/camera/rgbd</topic>
+                    <topic>${namespace}/camera/rgbd</topic>
                 </sensor>
             </gazebo>
